Commit message: update urdf and launch codes

File: rover_bot_description/description/part_macros.xacro (robot description, xacro)
@@ -145,4 +145,22 @@
         </collision>
         <xacro:inertial_box mass="0.2" x="${rocker_length}" y="0.05" z="0.02">
+            <origin xyz="0 0 0" rpy="0 0 0"/>
+        </xacro:inertial_box>
+    </xacro:macro>
+    <xacro:macro name="insert_stopper_link">
+        <visual>
+            <origin xyz="0 0 0" rpy="0 0 0"/>
+            <geometry>
+                <box size="0.1 0.05 0.02"/>
+            </geometry>
+            <material name="grey"/>
+        </visual>
+        <collision>
+            <origin xyz="0 0 0" rpy="0 0 0"/>
+            <geometry>
+                <box size="0.1 0.05 0.02"/>
+            </geometry>
+        </collision>
+        <xacro:inertial_box mass="0.2" x="0.1" y="0.05" z="0.02">
             <origin xyz="0 0 0" rpy="0 0 0"/>
         </xacro:inertial_box>

File: rover_bot_description/description/urdf_description.xacro (robot description, xacro)
@@ -49,5 +49,5 @@
     <xacro:arg name="imu_visual"   default="true"/>
     <xacro:arg name="sonar_visual"   default="false"/>
-    <xacro:arg name="cam_visual"   default="true"/>
+    <xacro:arg name="cam_visual"   default="false"/>
     <xacro:include filename="$(find rover_bot_description)/description/inertia_macros.xacro"/>
     <xacro:include filename="$(find rover_bot_description)/description/part_macros.xacro"/>
@@ -93,4 +93,17 @@
     </gazebo>
     <!--  ########################### -->
+    <!-- LEFT ROCKER STOPPER LINK -->
+    <!-- <joint name="left_rocker_stopper_joint" type="fixed">
+        <parent link="chassis_link"/>
+        <child link="left_rocker_stopper_link"/>
+        <origin xyz="${(rocker_length/2)-0.025} ${(chassis_width/2)+rocker_clearance} 0.05" rpy="0 0 0"/>
+    </joint>
+    <link name="left_rocker_stopper_link">
+        <xacro:insert_stopper_link/>
+    </link>
+    <gazebo reference="left_rocker_stopper_link">
+        <material>Gazebo/DarkGrey</material>
+    </gazebo> -->
+    <!--  ########################### -->
     <!-- LEFT ROCKER FRONT SERVO HINGE LINK -->
     <joint name="left_rocker_front_servo_hinge_joint" type="revolute">
@@ -176,4 +189,17 @@
         <material>Gazebo/DarkGrey</material>
     </gazebo>
+    <!--  ########################### -->
+    <!-- LEFT ROCKER STOPPER LINK -->
+    <!-- <joint name="right_rocker_stopper_joint" type="fixed">
+        <parent link="chassis_link"/>
+        <child link="right_rocker_stopper_link"/>
+        <origin xyz="${(rocker_length/2)-0.02} ${-1*((chassis_width/2)+rocker_clearance)} 0.05" rpy="0 0 0"/>
+    </joint>
+    <link name="right_rocker_stopper_link">
+        <xacro:insert_stopper_link/>
+    </link>
+    <gazebo reference="right_rocker_stopper_link">
+        <material>Gazebo/DarkGrey</material>
+    </gazebo> -->
     <!--  ########################### -->
     <!-- RIGHT ROCKER FRONT SERVO HINGE LINK -->
