Commit message: cleanup successfull

File: rover_bot_description/description/inertia_macros.xacro (robot description, xacro)
@@ -1,7 +1,4 @@
 <?xml version="1.0"?>
-<robot xmlns:xacro="http://www.ros.org/wiki/xacro" name="rover_bot">
-    <!-- Specify some standard inertial calculations https://en.wikipedia.org/wiki/List_of_moments_of_inertia -->
-    <!-- These make use of xacro's mathematical functionality -->
-    <!-- ################### inertia macros  ############################-->
+<robot xmlns:xacro="http://www.ros.org/wiki/xacro">
     <xacro:macro name="inertial_sphere" params="mass radius *origin">
         <inertial>
@@ -31,4 +28,3 @@
         </inertial>
     </xacro:macro>
-    <!-- ###################################################################################### -->
 </robot>

File: rover_bot_description/description/part_macros.xacro (robot description, xacro)
@@ -1,6 +1,5 @@
 <?xml version="1.0"?>
-<robot name="rover_bot" xmlns:xacro="http://www.ros.org/wiki/xacro" >
+<robot xmlns:xacro="http://www.ros.org/wiki/xacro" >
     <xacro:macro name="box_with_fillet" params="size_x size_y size_z fr material x y z">
-            <!-- logitudinal box -->
             <visual>
                 <origin xyz="${x} ${y} ${z}" rpy="0 0 0"/>
@@ -10,5 +9,4 @@
                 <material name="${material}"/>
             </visual>
-            <!-- lateral box -->
             <visual>
                 <origin xyz="${x} ${y} ${z}" rpy="0 0 0"/>
@@ -18,5 +16,4 @@
                 <material name="${material}"/>
             </visual>
-            <!-- cylinder1 -->
             <visual>
                 <origin xyz="${x+((size_x/2)-fr)} ${y+((size_y/2)-fr)} ${z}" rpy="0 0 0"/>
@@ -26,5 +23,4 @@
                 <material name="${material}"/>
             </visual>
-            <!-- cylinder2 -->
             <visual>
                 <origin xyz="${x+((size_x/2)-fr)} ${y-((size_y/2)-fr)} ${z}" rpy="0 0 0"/>
@@ -34,5 +30,4 @@
                 <material name="${material}"/>
             </visual>
-            <!-- cylinder3 -->
             <visual>
                 <origin xyz="${x-((size_x/2)-fr)} ${y+((size_y/2)-fr)} ${z}" rpy="0 0 0"/>
@@ -42,5 +37,4 @@
                 <material name="${material}"/>
             </visual>
-            <!-- cylinder4 -->
             <visual>
                 <origin xyz="${x-((size_x/2)-fr)} ${y-((size_y/2)-fr)} ${z}" rpy="0 0 0"/>

File: rover_bot_description/description/sensors/cam.xacro (robot description, xacro)
@@ -1,8 +1,6 @@
 <?xml version="1.0"?>
 <robot xmlns:xacro="http://www.ros.org/wiki/xacro"  name="rover_bot">
-    <!-- <xacro:arg name="cam_visual"   default="false"/> -->
     <xacro:property name="line_sense_angle"   value="${pi/2.5}"/>
     <xacro:property name="line_sense_mode"   value="true"/>
-    <!-- CAMERA LINK FRAME -->
     <joint name="cam_joint" type="fixed">
         <parent link="chassis_link"/>
@@ -69,12 +67,5 @@
             </camera>
             <plugin name="rgb_cam_plugin" filename="libgazebo_ros_camera.so">
-                <!-- <ros>
-                    <namespace>cam</namespace>
-                    <remapping>~/image_raw:=raw</remapping>
-                    <remapping>~/camera_info:=info</remapping>
-                </ros> -->
-                <!-- Set camera name. If empty, defaults to sensor name (i.e. "sensor_name") -->
                 <camera_name>cam</camera_name>
-                <!-- Set TF frame name. If empty, defaults to link name (i.e. "link_name") -->
                 <frame_name>cam_optical_link</frame_name>
                 <hack_baseline>0.2</hack_baseline>

File: rover_bot_description/description/sensors/imu.xacro (robot description, xacro)
@@ -1,6 +1,4 @@
 <?xml version="1.0"?>
 <robot xmlns:xacro="http://www.ros.org/wiki/xacro"  name="rover_bot">
-    <!-- <xacro:arg name="imu_visual"   default="true"/> -->
-  <!-- IMU LINK FRAME -->
     <joint name="imu_joint" type="fixed">
         <parent link="chassis_link"/>

File: rover_bot_description/description/sensors/lidar.xacro (robot description, xacro)
@@ -1,6 +1,4 @@
 <?xml version="1.0"?>
 <robot xmlns:xacro="http://www.ros.org/wiki/xacro"  name="rover_bot">
-    <!-- <xacro:arg name="laser_visual" default="false"/> -->
-    <!-- LIDAR LINK FRAME -->
     <joint name="lidar_joint" type="fixed">
         <parent link="chassis_link"/>

File: rover_bot_description/description/sensors/sonar.xacro (robot description, xacro)
@@ -1,8 +1,6 @@
 <?xml version="1.0"?>
 <robot xmlns:xacro="http://www.ros.org/wiki/xacro"  name="rover_bot">
-    <!-- <xacro:arg name="sonar_visual"   default="false"/> -->
     <xacro:property name="deg2rad" value="0.017460317"/>
     <xacro:property name="scan_angle" value="1"/>
-  <!-- SONAR LINK FRAME -->
     <joint name="sonar_joint" type="fixed">
         <parent link="chassis_link"/>

File: rover_bot_description/description/urdf_description.xacro (robot description, xacro)
@@ -29,13 +29,8 @@
     <xacro:property name="rocker_length" value="0.3"/>
     <xacro:property name="boggie_length" value="${(2*rocker_clearance)+chassis_width+0.05}"/>
-    <!-- WHEEL PARAMETERS -->
     <xacro:macro name="gazebo_wheel_settings" params="name">
         <gazebo reference="${name}">
             <mu1>1.0</mu1>
             <mu2>1.0</mu2>
-            <!-- <kp>${kp}</kp> -->
-            <!-- <kd>${kd}</kd> -->
-            <!-- <fdir1>${fdir}</fdir1> -->
-            <!-- <minDepth>${minDepth}</minDepth> -->
             <material>Gazebo/FlatBlack</material>
         </gazebo>
@@ -52,10 +47,6 @@
     <xacro:include filename="$(find rover_bot_description)/description/inertia_macros.xacro"/>
     <xacro:include filename="$(find rover_bot_description)/description/part_macros.xacro"/>
-    <!-- BASE LINK -->
-    <!-- <base joint/> -->
     <link name="base_link">
     </link>
-    <!-- ################# -->
-    <!-- CHASSIS LINK -->
     <joint name="chassis_joint" type="fixed">
         <parent link="base_link"/>
@@ -78,6 +69,4 @@
         <material>Gazebo/White</material>
     </gazebo>
-    <!--  ########################### -->
-    <!-- LEFT ROCKER LINK -->
     <joint name="left_rocker_joint" type="continuous">
         <parent link="chassis_link"/>
@@ -92,19 +81,4 @@
         <material>Gazebo/DarkGrey</material>
     </gazebo>
-    <!--  ########################### -->
-    <!-- LEFT ROCKER STOPPER LINK -->
-    <!-- <joint name="left_rocker_stopper_joint" type="fixed">
-        <parent link="chassis_link"/>
-        <child link="left_rocker_stopper_link"/>
-        <origin xyz="${(rocker_length/2)-0.025} ${(chassis_width/2)+rocker_clearance} 0.05" rpy="0 0 0"/>
-    </joint>
-    <link name="left_rocker_stopper_link">
-        <xacro:insert_stopper_link/>
-    </link>
-    <gazebo reference="left_rocker_stopper_link">
-        <material>Gazebo/DarkGrey</material>
-    </gazebo> -->
-    <!--  ########################### -->
-    <!-- LEFT ROCKER FRONT SERVO HINGE LINK -->
     <joint name="left_rocker_front_servo_hinge_joint" type="revolute">
         <parent link="left_rocker_link"/>
@@ -118,6 +92,4 @@
     </link>
     <xacro:gazebo_hinge_color name="left_rocker_front_servo_hinge_link"/>
-    <!--  ########################### -->
-    <!-- LEFT ROCKER FRONT WHEEL LINK -->
     <joint name="left_rocker_front_wheel_joint" type="continuous">
         <parent link="left_rocker_front_servo_hinge_link"/>
@@ -141,6 +113,4 @@
         <material>Gazebo/Red</material>
     </gazebo>
-    <!--  ########################### -->
-    <!-- LEFT ROCKER REAR SERVO HINGE LINK -->
     <joint name="left_rocker_rear_servo_hinge_joint" type="fixed">
         <parent link="left_rocker_link"/>
@@ -152,6 +122,4 @@
     </link>
     <xacro:gazebo_hinge_color name="left_rocker_rear_servo_hinge_link"/>
-    <!--  ########################### -->
-    <!-- LEFT ROCKER REAR WHEEL LINK -->
     <joint name="left_rocker_rear_wheel_joint" type="continuous">
         <parent link="left_rocker_rear_servo_hinge_link"/>
@@ -175,6 +143,4 @@
         <material>Gazebo/Red</material>
     </gazebo>
-    <!--  ########################### -->
-    <!-- RIGHT ROCKER LINK -->
     <joint name="right_rocker_joint" type="continuous">
         <parent link="chassis_link"/>
@@ -189,19 +155,4 @@
         <material>Gazebo/DarkGrey</material>
     </gazebo>
-    <!--  ########################### -->
-    <!-- LEFT ROCKER STOPPER LINK -->
-    <!-- <joint name="right_rocker_stopper_joint" type="fixed">
-        <parent link="chassis_link"/>
-        <child link="right_rocker_stopper_link"/>
-        <origin xyz="${(rocker_length/2)-0.02} ${-1*((chassis_width/2)+rocker_clearance)} 0.05" rpy="0 0 0"/>
-    </joint>
-    <link name="right_rocker_stopper_link">
-        <xacro:insert_stopper_link/>
-    </link>
-    <gazebo reference="right_rocker_stopper_link">
-        <material>Gazebo/DarkGrey</material>
-    </gazebo> -->
-    <!--  ########################### -->
-    <!-- RIGHT ROCKER FRONT SERVO HINGE LINK -->
     <joint name="right_rocker_front_servo_hinge_joint" type="revolute">
         <parent link="right_rocker_link"/>
@@ -215,6 +166,4 @@
     </link>
     <xacro:gazebo_hinge_color name="right_rocker_front_servo_hinge_link"/>
-    <!--  ########################### -->
-    <!-- RIGHT ROCKER FRONT WHEEL LINK -->
     <joint name="right_rocker_front_wheel_joint" type="continuous">
         <parent link="right_rocker_front_servo_hinge_link"/>
@@ -238,11 +187,8 @@
         <material>Gazebo/Red</material>
     </gazebo>
-    <!--  ########################### -->
-    <!-- RIGHT ROCKER REAR SERVO HINGE LINK -->
     <joint name="right_rocker_rear_servo_hinge_joint" type="fixed">
         <parent link="right_rocker_link"/>
         <child link="right_rocker_rear_servo_hinge_link"/>
         <origin xyz="${-1*((rocker_length/2)-0.025)} 0 -0.01" rpy="0 0 ${pi}"/>
-        <!-- <origin xyz="-0.145 0 -0.01" rpy="0 0 ${pi}"/> -->
     </joint>
     <link name="right_rocker_rear_servo_hinge_link">
@@ -250,6 +196,4 @@
     </link>
     <xacro:gazebo_hinge_color name="right_rocker_rear_servo_hinge_link"/>
-    <!--  ########################### -->
-    <!-- RIGHT ROCKER REAR WHEEL LINK -->
     <joint name="right_rocker_rear_wheel_joint" type="continuous">
         <parent link="right_rocker_rear_servo_hinge_link"/>
@@ -273,11 +217,8 @@
         <material>Gazebo/Red</material>
     </gazebo>
-    <!--  ########################### -->
-    <!-- BOGGIE LINK -->
     <joint name="boggie_joint" type="continuous">
         <parent link="chassis_link"/>
         <child link="boggie_link"/>
         <origin xyz="${-1*(rocker_length-0.05)} 0 0" rpy="0 0 0"/>
-        <!-- <origin xyz="-0.27 0 -0.01" rpy="0 0 0"/> -->
         <axis xyz="1 0 0"/>
     </joint>
@@ -288,6 +229,4 @@
         <material>Gazebo/DarkGrey</material>
     </gazebo>
-    <!--  ########################### -->
-    <!-- LEFT BOGGIE SERVO HINGE LINK -->
     <joint name="left_boggie_servo_hinge_joint" type="revolute">
         <parent link="boggie_link"/>
@@ -301,6 +240,4 @@
     </link>
     <xacro:gazebo_hinge_color name="left_boggie_servo_hinge_link"/>
-    <!--  ########################### -->
-    <!-- LEFT BOGGIE WHEEL LINK -->
     <joint name="left_boggie_wheel_joint" type="continuous">
         <parent link="left_boggie_servo_hinge_link"/>
@@ -324,6 +261,4 @@
         <material>Gazebo/Red</material>
     </gazebo>
-    <!--  ########################### -->
-    <!-- RIGHT BOGGIE SERVO HINGE LINK -->
     <joint name="right_boggie_servo_hinge_joint" type="revolute">
         <parent link="boggie_link"/>
@@ -337,6 +272,4 @@
     </link>
     <xacro:gazebo_hinge_color name="right_boggie_servo_hinge_link"/>
-    <!--  ########################### -->
-    <!-- RIGHT BOGGIE WHEEL LINK -->
     <joint name="right_boggie_wheel_joint" type="continuous">
         <parent link="right_boggie_servo_hinge_link"/>
@@ -360,5 +293,4 @@
         <material>Gazebo/Red</material>
     </gazebo>
-    <!--  ########################### -->
     <xacro:include filename="$(find rover_bot_description)/description/controllers.xacro"/>
     <xacro:include filename="$(find rover_bot_description)/description/sensors/imu.xacro"/>
